Commit message: fix(gamora): bind hardware arg to a property before comparing
${$(arg hardware) == 'mock'} expands to ${mock == 'mock'}, where mock is an
undefined name at xacro evaluation time. Binding the arg to a property first
gives a string to compare against. Verified by expanding the description with
xacro and parsing the result with check_urdf.

File: ros2/gamora_description/urdf/gamora_test_v6.urdf.xacro (robot description, xacro)
@@ -12,4 +12,5 @@
        "gazebo" swaps in the gz_ros2_control plugin. -->
   <xacro:arg name="hardware" default="mock"/>
+  <xacro:property name="hardware_type" value="$(arg hardware)"/>
   <xacro:arg name="initial_positions_file" default="$(find gamora_moveit_config)/config/initial_positions.yaml"/>
   <xacro:property name="initial_positions"
@@ -18,5 +19,5 @@
   <xacro:include filename="$(find gamora_description)/urdf/gamora_test_v6.urdf"/>
   <ros2_control name="GamoraSystem" type="system">
-    <xacro:if value="${$(arg hardware) == 'mock'}">
+    <xacro:if value="${hardware_type == 'mock'}">
       <hardware>
         <plugin>mock_components/GenericSystem</plugin>
@@ -24,5 +25,5 @@
       </hardware>
     </xacro:if>
-    <xacro:if value="${$(arg hardware) == 'gazebo'}">
+    <xacro:if value="${hardware_type == 'gazebo'}">
       <hardware>
         <plugin>gz_ros2_control/GazeboSimSystem</plugin>
@@ -48,5 +49,5 @@
     <xacro:joint_interfaces name="joint_reff"/>
   </ros2_control>
-  <xacro:if value="${$(arg hardware) == 'gazebo'}">
+  <xacro:if value="${hardware_type == 'gazebo'}">
     <gazebo>
       <plugin filename="gz_ros2_control-system"
